File: BelaMini_Amp/BelaMini_Amp.kicad_pcb (KiCad board)
At the start: 2 copper layers, 83.8 x 73.7 mm, 46 parts, among them J1 OUT_L, J2 OUT_R, J3 Conn_01x03_Female, J4 Conn_01x03_Female, SW1 SW_Push, SW2 SW_Push, SW3 SW_Push, U1 BelaMini, U2 TPA2016D2RTJR

Commit message: Updated example
Parts:
- removed the REF** at (88.3, 55.2)
- removed the REF** at (88.3, 118.7)
- removed the REF** at (161.9, 118.7)
- removed the REF** at (161.9, 55.2)
- added G***: LOGO, AIL_Kicad_Workshop:AIL_logo, F.Cu at (123.2, 76.2)
- added REF**: MountingHole_3.2mm_M3_Pad_Via, MountingHole:MountingHole_3.2mm_M3_Pad_Via, F.Cu at (190.5, 68.6)
- added REF**: MountingHole_3.2mm_M3_Pad_Via, MountingHole:MountingHole_3.2mm_M3_Pad_Via, F.Cu at (116.8, 68.6)
- added REF**: MountingHole_3.2mm_M3_Pad_Via, MountingHole:MountingHole_3.2mm_M3_Pad_Via, F.Cu at (116.8, 132.1)
- added REF**: MountingHole_3.2mm_M3_Pad_Via, MountingHole:MountingHole_3.2mm_M3_Pad_Via, F.Cu at (190.5, 132.1)
- added RV3: R_POT, Potentiometer_THT:Potentiometer_Alpha_RD901F-40-00D_Single_Vertical, F.Cu at (178.4, 80.6)
- moved RV2 35.5 mm to (178.4, 97.2)
- moved C1 31.5 mm to (157.1, 77.3)
- moved C2 31.5 mm to (157.1, 80.6)
- moved SW3 31.5 mm to (173.1, 133.2)
- moved C12 31.5 mm to (166.4, 68.5)
- moved C13 31.5 mm to (164.5, 68.5)
- moved C8 31.5 mm to (146.1, 78.9)
- moved D2 31.5 mm to (150.2, 103.5)
- moved D3 31.5 mm to (165.2, 103.5)
- moved FB2 31.5 mm to (157.1, 78.9)
- moved R4 31.5 mm to (151.6, 108.6)
- moved R8 31.5 mm to (166.5, 108.6)
- moved C10 31.5 mm to (138.4, 68.5)
- moved C11 31.5 mm to (140.3, 68.5)
- moved C6 31.5 mm to (148.8, 83.3)
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Connections:
- U1 pad A2: Net-(U1-PadA2) -> /A2
Routing:
- net /A2: track 0.00 -> 35.6 mm
- net 5V: track 105.9 -> 118.9 mm
- net /A1: track 25.9 -> 18.0 mm
- net /A0: track 7.25 -> 6.62 mm
- net GND: vias 13 -> 15
- added copper zone on F.Cu, net Net-(C10-Pad1)
- added copper zone on F.Cu, net Net-(C11-Pad1)
- added copper zone on F.Cu, net Net-(C12-Pad1)
- added copper zone on F.Cu, net Net-(C13-Pad1)
Other:
- board text added: "2.8W Stereo [4-8 ohm]"
- board text added: "IN"
- board text added: "June/2020"
- board text added: "LEFT"
- board text added: "OUT"
- board text added: "RIGHT"
- board text added: "TPA2016"
- board text added: "rev 1.0"
